File: Hardware/ebook-reader v156.sch (EAGLE design)
At the start: 103 parts, among them IC1 BD5229G-TR, IC4 XC6220A331MR-G, J1 FH34SRJ-24S-0.5SH_99_, J2 SAMACSYS_PARTS_USB4110-GF-A, J3 QWIIC_RIGHT_ANGLE, J4 112A-TAAR-R03_ATTEND, Q1 20V/4.2A/52mΩ/1.4W, Q2 20V/4.2A/52mΩ/1.4W, Q3 SI1308EDL-T1-GE3, U1 W25Q512JVEIQ, U2 ESP32-C6-WROOM-1-N8, U3 DS3231SN#, U4 MAX17048G+T10

Commit message: add final .sch and .brd final versions
Parts:
- C3: value 100uF -> 100uF TANT
- CHG_LED: value (none) -> &
- R10, R5, R6, R7, R8, R9: value (none) -> 10K
- SJ1: value (none) -> T
Connections:
- net N$3 renamed GPIO8
- new net N$3: EPD_C11.2, J1.23
- net GND: now also EPD_C10.1, EPD_C11.1, EPD_C12.1, EPD_C5.1, EPD_C6.1, EPD_C7.1, EPD_C8.1, EPD_C9.2
- net N$1: no longer J2.A8
- net N$17: no longer EPD_C11.2, J1.23
- net PREVGL: no longer EPD_C10.1, EPD_C11.1, EPD_C12.1, EPD_C5.1, EPD_C6.1, EPD_C7.1, EPD_C8.1, EPD_C9.2
Other:
- note added: "OpenBook Schematic"
- note removed: "ebook-reader"
